File: hardware/pt-thrifty/pt_thrifty.kicad_sch (KiCad schematic)
At the start: 23 parts, among them J1 Conn_01x09, J2 Conn_01x09, J3 SJ-43514-SMT-TR, SW1 PTS636 SM50J SMTR LFS, SW2 SW_Push_Shielded, U2 MCP6273T-E/CH

Commit message: WIP pt-thrifty rev3 sch/pcb
Parts:
- removed C6: 100nF, Capacitor_SMD:C_0603_1608Metric, symbol Device:C
- removed R8, R9: 22R, Resistor_SMD:R_0603_1608Metric, symbol Device:R
- removed SW1: PTS636 SM50J SMTR LFS, PicoTimecode_PCB_Rev2:SW_PTS636_CNK, symbol 2024-11-18_16-32-35:PTS636_SM50J_SMTR_LFS
- added J4: Conn_01x08, Connector_PinSocket_2.54mm:PinSocket_1x08_P2.54mm_Vertical, symbol Connector_Generic:Conn_01x08
- added R1, R14, R2: 100R, Resistor_SMD:R_0603_1608Metric, symbol Device:R
- added R10, R11, R12, R13: 100K, Resistor_SMD:R_0603_1608Metric, symbol Device:R
- added TP1: TestPoint, TestPoint:TestPoint_THTPad_1.0x1.0mm_Drill0.5mm, symbol Connector:TestPoint
- added U3: MCP6273T-E/CH, Package_TO_SOT_SMD:SOT-23-6, symbol 2024-12-04_21-34-14:MCP6273T-E_CH
- C1, C5: value 100nF -> 1uF
- C2: value 100nF -> 1uF; now not fitted
- R3: renamed from R1; value 10K -> 100K
- R4: renamed from R2; value 10K -> 100K
- R5: renamed from R3; value 10K -> 2.00K-1%
- R6: renamed from R4; value 10K -> 2.00K-1%
- R8: renamed from R5; value 2.10K-1% -> 2.00K-1%
- R9: renamed from R6; value 2.00K-1% -> 2.49K-1%
- SW1: renamed from SW2; now not fitted
- U1: value ~ -> (none)
Connections:
- net +3.3V: now also C5.2, J4.2 (Pin_2), U3.6 (VDD)
- net GND: now also C5.1, R4.2, R6.2, J4.1 (Pin_1), J4.8 (Pin_8), R11.2, U3.2 (VSS)
- net IN_OUT_L: now also R1.2; no longer C5.1
- net IN_OUT_R: now also R2.2
- net VREF: now also R12.1
- net ROT_SW: now reaches U1.15 (GPIO29)
- net ROT_SW: now also J2.4 (Pin_4)
- net CLAP_SW: now reaches J2.5 (Pin_5)
- net CLAP_SW: now also U1.14 (GPIO28)
- net SPI0_RST: now reaches J2.7 (Pin_7), U1.12 (GPIO26)
- net SPI0_RST: now also J4.5 (Pin_5)
- net I2C1_SCLK: now reaches J2.8 (Pin_8), U1.11 (GPIO15)
- net I2C1_SDA: now reaches J2.9 (Pin_9), U1.10 (GPIO14)
- net at R8.2, R9.2: now also R10.1; no longer C5.2
- net SPI0_DC: now reaches J1.5 (Pin_5), U1.5 (GPIO4)
- net SPI0_DC: now also J4.6 (Pin_6)
- net SPI0_CSn: now reaches J1.6 (Pin_6), U1.6 (GPIO5)
- net SPI0_CSn: now also J4.7 (Pin_7)
- net SPI0_SCK: now reaches J1.7 (Pin_7), U1.7 (GPIO6)
- net SPI0_SCK: now also J4.3 (Pin_3)
- net SPI0_TX: now reaches J1.8 (Pin_8), U1.8 (GPIO7)
- net SPI0_TX: now also J4.4 (Pin_4)
- net AMP_nEN1: now reaches J1.9 (Pin_9), U1.9 (GPIO8)
- net AMP_nEN1: now also R14.2
- net AMP_CS renamed AMP_nEN0
- net AMP_nEN0: no longer R4.2, R6.2
- new net: R10.2, R11.1, U3.3 (VIN+)
- new net: R14.1, U3.5 (*CS)
- new net: R12.2, R13.1, U3.4 (VIN-)
- new net OUTPUT: R1.1, R13.2, R2.1, TP1.1, U3.1 (VOUT)
Other:
- added sheet sony_mi (sony_mi.kicad_sch)
- added sheet time-bar (time-bar.kicad_sch)
- note added: "(extra)"
- note added: "2026-07-28 © Simon Wood"
- note added: "D0"
- note added: "D1"
- note added: "Just for Routing"
- note added: "LTC Interface for WaveShare RP2040-Zero"
- note added: "Note: Differential Drive will produce ~100mV pk-pk signal. Force nLTC_TX high for ~1V pk-pk signal."
- note added: "Rev 3"
- note added: "SSD1366 OLED Display (7-pin)"
- note added: "Select which channel to output on..."
- note added: "Select which channel to receive on..."
- note removed: "2025-12-04 © Simon Wood"
- note removed: "Note: Bottom of dividers connected to nCS, this needs to be driven low to enable RX amplifier. Float/Pull-up for PowerSave"
- note removed: "Note: Differential Drive will produce ~80mV pk-pk signal. Force nLTC_TX low for ~1V pk-pk signal."
- note removed: "Rev 2"
- moved on the sheet: C1, C3, C4, J1, J2, J3, LED1, R3, R4, R5, R6, R7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

Commit message: Clean up the Kicad files for PT-Thrifty
Parts:
- removed LED1: LTST-S220GKT, footprints:LED_LTST-S220GKT_LTO, symbol 2024-02-24_16-38-46:LTST-S220GKT
- removed U2, U3: MCP6273T-E/CH, Package_TO_SOT_SMD:SOT-23-6, symbol 2024-12-04_21-34-14:MCP6273T-E_CH
- added LED1: LTST-S220GKT, LED_LTST-S220GKT_LTO, symbol LTST_S220GKT:LTST-S220GKT
- added U2, U3: MCP6273T-E/CH, SOT-23-6_MC_MCH, symbol MCP6273T_E_CH:MCP6273T-E_CH
- J3: footprint PicoTimecode_PCB_Rev2:CUI_SJ-43514-SMT-TR -> CUI_SJ-43514-SMT-TR
Connections:
- net +3.3V: now also U2.6 (VDD), U3.6 (VDD)
- net AMP_nEN0: now also U2.5 (*CS)
- net GND: now also LED1.1, U2.2 (VSS), U3.2 (VSS)
- net IN: now also U2.3 (VIN+)
- net LTX_RX: now also U2.1 (VOUT)
- net OUTPUT: now also U3.1 (VOUT)
- net VREF: now also U2.4 (VIN-)
- net at R7.2: now also LED1.2
- net at R10.2, R11.1: now also U3.3 (VIN+)
- net at R14.1: now also U3.5 (*CS)
- net at R12.2, R13.1: now also U3.4 (VIN-)

Commit message: Re-import symbols into PCB layout
Parts:
- J3: footprint CUI_SJ-43514-SMT-TR -> SJ-43514-SMT-TR:CUI_SJ-43514-SMT-TR
- LED1: footprint LED_LTST-S220GKT_LTO -> LTST_S220GKT:LED_LTST-S220GKT_LTO
- U2, U3: footprint SOT-23-6_MC_MCH -> MCP6273T_E_CH:SOT-23-6_MC_MCH-L
Changed lines of the file:
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@@
 			)
 		)
-		(property "Footprint" "CUI_SJ-43514-SMT-TR"
+		(property "Footprint" "SJ-43514-SMT-TR:CUI_SJ-43514-SMT-TR"
 			(at 60.96 116.84 0)
 			(hide yes)
@@
 			)
 		)
-		(property "Footprint" "SOT-23-6_MC_MCH"
+		(property "Footprint" "MCP6273T_E_CH:SOT-23-6_MC_MCH-L"
 			(at 215.9 144.78 0)
 			(hide yes)
@@
 			)
 		)
-		(property "Footprint" "LED_LTST-S220GKT_LTO"
+		(property "Footprint" "LTST_S220GKT:LED_LTST-S220GKT_LTO"
 			(at 62.23 172.72 0)
 			(hide yes)
@@
 			)
 		)
-		(property "Footprint" "SOT-23-6_MC_MCH"
+		(property "Footprint" "MCP6273T_E_CH:SOT-23-6_MC_MCH-L"
 			(at 187.96 90.17 0)
 			(hide yes)

Commit message: Add 3D models and pin-1 markings
Parts:
- LED1: footprint LTST_S220GKT:LED_LTST-S220GKT_LTO -> LTST_S220GKT:LED_LTST-S220GKT_LTO-L
Changed lines of the file:
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@@
 			)
 		)
-		(property "Footprint" "LTST_S220GKT:LED_LTST-S220GKT_LTO"
+		(property "Footprint" "LTST_S220GKT:LED_LTST-S220GKT_LTO-L"
 			(at 62.23 172.72 0)
 			(hide yes)
